File: OpenLTTO Sensor Module.kicad_sch (KiCad schematic)
At the start: 6 parts

Commit message: Updated schematic metadata, added schematic PDF, and PCB Renders
Other:
- company: (none) -> Paul Mumby
- title: (none) -> OpenLTTO Sensor Module
Changed lines of the file:
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@@
 (kicad_sch (version 20230121) (generator eeschema)
   (paper "A4")
+  (title_block
+    (title "OpenLTTO Sensor Module")
+    (rev "1.0")
+    (company "Paul Mumby")
+  )
   (junction (at 163.83 85.09) (diameter 0) (color 0 0 0 0)
   )
