File: ir_module.kicad_sch (KiCad schematic)
At the start: 8 parts, among them Q1 IRLML6244, U1 TSOP4138

Commit message: Updated schematic metadata, added schematic PDF, and PCB Renders
Other:
- company: (none) -> Paul Mumby
- title: (none) -> OpenLTTO Sensor Module
Changed lines of the file:
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@@
 (kicad_sch (version 20230121) (generator eeschema)
   (paper "A4")
+  (title_block
+    (title "OpenLTTO Sensor Module")
+    (rev "1.0")
+    (company "Paul Mumby")
+  )
   (junction (at 152.4 106.68) (diameter 0) (color 0 0 0 0)
   )
